Commit message: Updated files from other simulatori

File: simple_arm/urdf/panda.ros2_control.xacro (robot description, xacro)
@@ -4,7 +4,7 @@
         <xacro:property name="initial_positions" value="${load_yaml(initial_positions_file)['initial_positions']}"/>
         <ros2_control name="${name}" type="system">
-            <hardware>
-                <plugin>gazebo_ros2_control/GazeboSystem</plugin>
-            </hardware>
+        <hardware>
+            <plugin>ignition_ros2_control/IgnitionSystem</plugin>
+        </hardware>
             <joint name="panda_joint1">
                 <param name="initial_position">${initial_positions['panda_joint1']}</param>

File: simple_arm/urdf/panda_gazebo.urdf.xacro (robot description, xacro)
@@ -59,19 +59,19 @@
         <xacro:arm_control transmission="${arm_id}_rightfinger" joint="${arm_id}_finger_joint2" motor="${arm_id}_finger_joint2"/>
     </xacro:macro>
-  <link name="world"/>
-  <joint name="panda_to_world" type="fixed">
-    <parent link="world"/>
-    <child link="panda_link0"/>
-    <origin rpy="0 0 0" xyz="0 0 0"/>
-    <dynamics damping="1.0"/>
-  </joint>
-<xacro:panda_gazebo arm_id="panda"/>
+    <link name="world"/>
+    <joint name="panda_to_world" type="fixed">
+        <parent link="world"/>
+        <child link="panda_link0"/>
+        <origin rpy="0 0 0" xyz="0 0 0"/>
+        <dynamics damping="1.0"/>
+    </joint>
+    <xacro:panda_gazebo arm_id="panda"/>
   <!-- <xacro:panda_control arm_id="panda"/> -->
-  <gazebo>
-    <plugin filename="libgazebo_ros2_control.so" name="gazebo_ros2_control">
-      <robot_param>robot_description</robot_param>
-      <robot_param_node>robot_state_publisher</robot_param_node>
-      <parameters>$(find simple_arm)/config/panda_ros_controllers.yaml</parameters>
-    </plugin>
-  </gazebo>
+    <gazebo>
+        <plugin filename="libignition_ros2_control.so" name="ignition_ros2_control">
+        <robot_param>robot_description</robot_param>
+        <robot_param_node>robot_state_publisher</robot_param_node>
+        <parameters>$(find ignition_ros2_control_demos)/config/cartpole_controller.yaml</parameters>
+        </plugin>
+    </gazebo>
 </robot>

File: simple_arm/urdf/panda_hand.ros2_control.xacro (robot description, xacro)
@@ -4,5 +4,5 @@
         <ros2_control name="${name}" type="system">
             <hardware>
-                <plugin>gazebo_ros2_control/GazeboSystem</plugin>
+                <plugin>ignition_ros2_control/IgnitionSystem</plugin>
             </hardware>
             <joint name="panda_finger_joint1">
@@ -13,6 +13,4 @@
             </joint>
             <joint name="panda_finger_joint2">
-                <param name="mimic">panda_finger_joint1</param>
-                <param name="multiplier">1</param>
                 <command_interface name="position" />
                 <state_interface name="position"/>
