Commit message: Working moveit implementation

File: simple_arm/urdf/panda.urdf.xacro (robot description, xacro)
@@ -11,14 +11,18 @@
         <xacro:macro name="arm_gazebo" params="link">
             <gazebo reference="${link}">
-                <material>Gazebo/White</material>
-                <mu1>0.2</mu1>
-                <mu2>0.2</mu2>
+                <material>
+                    <ambient> 1 1 1 1</ambient>
+                    <diffuse> 1 1 1 1</diffuse>
+                    <specular> .1 .1 .1 128</specular>
+                </material>
             </gazebo>
         </xacro:macro>
         <xacro:macro name="hand_gazebo" params="link">
             <gazebo reference="${link}">
-                <material>Gazebo/Grey</material>
-                <mu1>0.2</mu1>
-                <mu2>0.2</mu2>
+                <material>
+                    <ambient> .3 .3 .3  1.0</ambient>
+                    <diffuse> .7 .7 .7  1.0</diffuse>
+                    <specular> 0.01 0.01 0.01 1.000000 1.500000</specular>
+                </material>
             </gazebo>
         </xacro:macro>
@@ -36,27 +40,4 @@
         <xacro:hand_gazebo link="${arm_id}_leftfinger"/>
     </xacro:macro>
-    <xacro:macro name="panda_control" params="arm_id">
-        <xacro:macro name="arm_control" params="transmission joint motor">
-            <transmission name="${transmission}">
-                <type>transmission_interface/SimpleTransmission</type>
-                <joint name="${joint}">
-                    <hardwareInterface>hardware_interface/PositionJointInterface</hardwareInterface>
-                </joint>
-                <actuator name="${motor}">
-                    <hardwareInterface>hardware_interface/PositionJointInterface</hardwareInterface>
-                    <mechanicalReduction>1</mechanicalReduction>
-                </actuator>
-            </transmission>
-        </xacro:macro>
-        <xacro:arm_control transmission="${arm_id}_tran_1" joint="${arm_id}_joint1" motor="${arm_id}_motor_1"/>
-        <xacro:arm_control transmission="${arm_id}_tran_2" joint="${arm_id}_joint2" motor="${arm_id}_motor_2"/>
-        <xacro:arm_control transmission="${arm_id}_tran_3" joint="${arm_id}_joint3" motor="${arm_id}_motor_3"/>
-        <xacro:arm_control transmission="${arm_id}_tran_4" joint="${arm_id}_joint4" motor="${arm_id}_motor_4"/>
-        <xacro:arm_control transmission="${arm_id}_tran_5" joint="${arm_id}_joint5" motor="${arm_id}_motor_5"/>
-        <xacro:arm_control transmission="${arm_id}_tran_6" joint="${arm_id}_joint6" motor="${arm_id}_motor_6"/>
-        <xacro:arm_control transmission="${arm_id}_tran_7" joint="${arm_id}_joint7" motor="${arm_id}_motor_7"/>
-        <xacro:arm_control transmission="${arm_id}_leftfinger" joint="${arm_id}_finger_joint1" motor="${arm_id}_finger_joint1"/>
-        <xacro:arm_control transmission="${arm_id}_rightfinger" joint="${arm_id}_finger_joint2" motor="${arm_id}_finger_joint2"/>
-    </xacro:macro>
     <link name="world"/>
     <joint name="panda_to_world" type="fixed">
@@ -67,5 +48,5 @@
     </joint>
     <xacro:panda_gazebo arm_id="panda"/>
-  <!-- <xacro:panda_control arm_id="panda"/> -->
+    <!-- <xacro:panda_control arm_id="panda"/> -->
     <gazebo>
     <plugin filename="ignition_ros2_control-system" name="ignition_ros2_control::IgnitionROS2ControlPlugin">
@@ -75,3 +56,4 @@
         </plugin>
     </gazebo>
+    <gravity>0 0 -9.8</gravity>
 </robot>

Commit message: Updated world and removed gazebo control

File: simple_arm/urdf/panda.urdf.xacro (robot description, xacro)
@@ -8,36 +8,4 @@
     <xacro:panda_ros2_control name="PandaGazeboControl" initial_positions_file="$(arg initial_positions_file)"/>
     <xacro:panda_hand_ros2_control name="PandaHandGazeboControl"/>
-    <xacro:macro name="panda_gazebo" params="arm_id">
-        <xacro:macro name="arm_gazebo" params="link">
-            <gazebo reference="${link}">
-                <material>
-                    <ambient> 1 1 1 1</ambient>
-                    <diffuse> 1 1 1 1</diffuse>
-                    <specular> .1 .1 .1 128</specular>
-                </material>
-            </gazebo>
-        </xacro:macro>
-        <xacro:macro name="hand_gazebo" params="link">
-            <gazebo reference="${link}">
-                <material>
-                    <ambient> .3 .3 .3  1.0</ambient>
-                    <diffuse> .7 .7 .7  1.0</diffuse>
-                    <specular> 0.01 0.01 0.01 1.000000 1.500000</specular>
-                </material>
-            </gazebo>
-        </xacro:macro>
-        <xacro:arm_gazebo link="${arm_id}_link0"/>
-        <xacro:arm_gazebo link="${arm_id}_link1"/>
-        <xacro:arm_gazebo link="${arm_id}_link2"/>
-        <xacro:arm_gazebo link="${arm_id}_link3"/>
-        <xacro:arm_gazebo link="${arm_id}_link4"/>
-        <xacro:arm_gazebo link="${arm_id}_link5"/>
-        <xacro:arm_gazebo link="${arm_id}_link6"/>
-        <xacro:hand_gazebo link="${arm_id}_link7"/>
-        <xacro:hand_gazebo link="${arm_id}_link8"/>
-        <xacro:hand_gazebo link="${arm_id}_hand"/>
-        <xacro:hand_gazebo link="${arm_id}_rightfinger"/>
-        <xacro:hand_gazebo link="${arm_id}_leftfinger"/>
-    </xacro:macro>
     <link name="world"/>
     <joint name="panda_to_world" type="fixed">
@@ -47,5 +15,4 @@
         <dynamics damping="1.0"/>
     </joint>
-    <xacro:panda_gazebo arm_id="panda"/>
     <!-- <xacro:panda_control arm_id="panda"/> -->
     <gazebo>
